Commit message: Log robot camera in Rerun

File: src/sam_bot_nav2_gz/src/description/sam_bot_description.urdf (robot description, URDF)
Before this commit: robot sam_bot, 7 links, 6 joints
Links:
- removed link camera_depth_frame
- added link camera_frame
Joints:
- removed joint camera_depth_joint
- added joint camera_frame_joint: type fixed, parent camera_link, child camera_frame, origin xyz=0 0 0 rpy=${-pi/2} 0 ${-pi/2}

Commit message: GNSS based navigation.

File: src/sam_bot_nav2_gz/src/description/sam_bot_description.urdf (robot description, URDF)
Before this commit: robot sam_bot, 7 links, 6 joints
Links:
- added link gnss_link; collision box size=0.1 0.1 0.1; visual box size=0.1 0.1 0.1
Joints:
- added joint gnss_joint: type fixed, parent base_link, child gnss_link, origin xyz=0 0 0.01
