Commit message: Works :) yay. But IMU is straight.

File: urdf/robot.xacro.urdf (robot description, URDF)
Before this commit: robot diff_drive, 7 links, 6 joints
Joints:
- joint gnss_joint: origin xyz=0.554282 0 1.5 rpy=0.3 1.6 -0.4 -> xyz=0.554282 0 1.5 rpy=0 0 0
- joint imu_joint: origin xyz=0.554283 0 1.0 rpy=-0.1 0.3 -1.77 -> xyz=0.554283 0 1.0 rpy=0 0 0
